File: hardware/atmega328p.sch (KiCad schematic (older format))
At the start: 17 parts, among them J401 USART, U401 ATMEGA328P-PU, Y401 16MHz

Commit message: Layout MT19 criado para o Taquímetro do barco.
Connections:
- net VOUT: now reaches U401.4 (PD2)
- no-connect marks 9 -> 8
Changed lines of the file:
@@
 EESchema Schematic File Version 4
 LIBS:basicsensormodule-cache
-EELAYER 26 0
+EELAYER 29 0
 EELAYER END
 $Descr A4 11693 8268
 encoding utf-8
-Sheet 3 5
+Sheet 3 6
 Title ""
 Date ""
@@
 NoConn ~ 5050 3950
 NoConn ~ 5050 4750
-NoConn ~ 5050 4650
 NoConn ~ 5050 4850
 Text Notes 5100 6400 0    60   ~ 0
@@
 Wire Wire Line
 	4950 4850 5050 4850
-Wire Wire Line
-	5050 4650 4950 4650
 Wire Wire Line
 	5050 4750 4950 4750
@@
 SDA
 NoConn ~ 5050 3650
+Text HLabel 5050 4650 2    50   Input ~ 0
+VOUT
+Wire Wire Line
+	4950 4650 5050 4650
 $EndSCHEMATC
