File: hardware/_autosave-basicsensormodule.kicad_pcb (KiCad board)
At the start: 2 copper layers, 52.1 x 121.3 mm, 63 parts, among them J1 Conn_01x04, J401 USART, J601 RJ45, J602 RJ45, U201 MCP2551-I/SN, U202 MCP2515-xSO, U301 A1101ELHL, U401 ATMEGA328P-PU, U501 LM7805, Y201 16MHz, Y401 16MHz

Commit message: Atualização MT19
Parts:
- moved C102 5.08 mm to (91.8, 47.6)
- moved J1 1.27 mm to (98.4, 44.5)
- moved TP204 1.27 mm to (70.5, 116.8)
Routing:
- net /CANBUS/RXCAN: track 16.0 -> 15.5 mm
- net +5V: track 209.8 -> 209.3 mm
- net /MCU/SDA: track 25.2 -> 25.7 mm
- net /MCU/SCL: track 22.0 -> 22.5 mm

Commit message: Atualização pdf MT19
Parts:
- added C1: 4.7n, Capacitor_SMD:C_0805_2012Metric_Pad1.15x1.40mm_HandSolder, B.Cu at (239.0, 50.8)
- added C1: 4.7n, Capacitor_SMD:C_0805_2012Metric_Pad1.15x1.40mm_HandSolder, B.Cu at (176.6, 50.8)
- added C1: 4.7n, Capacitor_SMD:C_0805_2012Metric_Pad1.15x1.40mm_HandSolder, B.Cu at (114.2, 50.8)
- added C101: 100n, Capacitor_SMD:C_0805_2012Metric_Pad1.15x1.40mm_HandSolder, B.Cu at (235.2, 39.4)
- added C101: 100n, Capacitor_SMD:C_0805_2012Metric_Pad1.15x1.40mm_HandSolder, B.Cu at (172.8, 39.4)
- added C101: 100n, Capacitor_SMD:C_0805_2012Metric_Pad1.15x1.40mm_HandSolder, B.Cu at (110.4, 39.4)
- added C102: 100nF, Capacitor_SMD:C_0805_2012Metric_Pad1.15x1.40mm_HandSolder, B.Cu at (248.6, 41.9)
- added C102: 100nF, Capacitor_SMD:C_0805_2012Metric_Pad1.15x1.40mm_HandSolder, B.Cu at (186.2, 41.9)
- added C102: 100nF, Capacitor_SMD:C_0805_2012Metric_Pad1.15x1.40mm_HandSolder, B.Cu at (123.8, 41.9)
- added C201: 100nF, Capacitor_SMD:C_0805_2012Metric_Pad1.15x1.40mm_HandSolder, B.Cu at (234.8, 97.2)
- added C201: 100nF, Capacitor_SMD:C_0805_2012Metric_Pad1.15x1.40mm_HandSolder, B.Cu at (172.4, 97.2)
- added C201: 100nF, Capacitor_SMD:C_0805_2012Metric_Pad1.15x1.40mm_HandSolder, B.Cu at (110.0, 97.2)
- added C202: 100nF, Capacitor_SMD:C_0805_2012Metric_Pad1.15x1.40mm_HandSolder, B.Cu at (242.4, 113.0)
- added C202: 100nF, Capacitor_SMD:C_0805_2012Metric_Pad1.15x1.40mm_HandSolder, B.Cu at (180.0, 113.0)
- added C202: 100nF, Capacitor_SMD:C_0805_2012Metric_Pad1.15x1.40mm_HandSolder, B.Cu at (117.6, 113.0)
- added C203: 22pF, Capacitor_SMD:C_0805_2012Metric_Pad1.15x1.40mm_HandSolder, B.Cu at (227.2, 103.3)
- added C203: 22pF, Capacitor_SMD:C_0805_2012Metric_Pad1.15x1.40mm_HandSolder, B.Cu at (164.8, 103.3)
- added C203: 22pF, Capacitor_SMD:C_0805_2012Metric_Pad1.15x1.40mm_HandSolder, B.Cu at (102.4, 103.3)
- added C204: 22pF, Capacitor_SMD:C_0805_2012Metric_Pad1.15x1.40mm_HandSolder, B.Cu at (229.4, 99.4)
- added C204: 22pF, Capacitor_SMD:C_0805_2012Metric_Pad1.15x1.40mm_HandSolder, B.Cu at (167.0, 99.4)
- added C204: 22pF, Capacitor_SMD:C_0805_2012Metric_Pad1.15x1.40mm_HandSolder, B.Cu at (104.6, 99.4)
- added C205: 100nF, Capacitor_SMD:C_0805_2012Metric_Pad1.15x1.40mm_HandSolder, B.Cu at (237.6, 122.9)
- added C205: 100nF, Capacitor_SMD:C_0805_2012Metric_Pad1.15x1.40mm_HandSolder, B.Cu at (175.2, 122.9)
- added C205: 100nF, Capacitor_SMD:C_0805_2012Metric_Pad1.15x1.40mm_HandSolder, B.Cu at (112.8, 122.9)
- added C401: 100nF, Capacitor_SMD:C_0805_2012Metric_Pad1.15x1.40mm_HandSolder, B.Cu at (245.9, 76.6)
- added C401: 100nF, Capacitor_SMD:C_0805_2012Metric_Pad1.15x1.40mm_HandSolder, B.Cu at (183.5, 76.6)
- added C401: 100nF, Capacitor_SMD:C_0805_2012Metric_Pad1.15x1.40mm_HandSolder, B.Cu at (121.1, 76.6)
- added C402: 100nF, Capacitor_SMD:C_0805_2012Metric_Pad1.15x1.40mm_HandSolder, B.Cu at (230.6, 71.5)
- added C402: 100nF, Capacitor_SMD:C_0805_2012Metric_Pad1.15x1.40mm_HandSolder, B.Cu at (168.2, 71.5)
- added C402: 100nF, Capacitor_SMD:C_0805_2012Metric_Pad1.15x1.40mm_HandSolder, B.Cu at (105.8, 71.5)
- added C403: 22pF, Capacitor_SMD:C_0805_2012Metric_Pad1.15x1.40mm_HandSolder, B.Cu at (228.1, 79.1)
- added C403: 22pF, Capacitor_SMD:C_0805_2012Metric_Pad1.15x1.40mm_HandSolder, B.Cu at (165.7, 79.1)
- added C403: 22pF, Capacitor_SMD:C_0805_2012Metric_Pad1.15x1.40mm_HandSolder, B.Cu at (103.3, 79.1)
- added C404: 22pF, Capacitor_SMD:C_0805_2012Metric_Pad1.15x1.40mm_HandSolder, B.Cu at (229.4, 74.7)
- added C404: 22pF, Capacitor_SMD:C_0805_2012Metric_Pad1.15x1.40mm_HandSolder, B.Cu at (167.0, 74.7)
- added C404: 22pF, Capacitor_SMD:C_0805_2012Metric_Pad1.15x1.40mm_HandSolder, B.Cu at (104.6, 74.7)
- added C405: 100nF, Capacitor_SMD:C_0805_2012Metric_Pad1.15x1.40mm_HandSolder, B.Cu at (229.4, 56.3)
- added C405: 100nF, Capacitor_SMD:C_0805_2012Metric_Pad1.15x1.40mm_HandSolder, B.Cu at (167.0, 56.3)
- added C405: 100nF, Capacitor_SMD:C_0805_2012Metric_Pad1.15x1.40mm_HandSolder, B.Cu at (104.6, 56.3)
- added C406: 100nF, Capacitor_SMD:C_0805_2012Metric_Pad1.15x1.40mm_HandSolder, B.Cu at (231.8, 51.3)
- added C406: 100nF, Capacitor_SMD:C_0805_2012Metric_Pad1.15x1.40mm_HandSolder, B.Cu at (169.4, 51.3)
- added C406: 100nF, Capacitor_SMD:C_0805_2012Metric_Pad1.15x1.40mm_HandSolder, B.Cu at (107.0, 51.3)
- added C501: 1uF, Capacitor_Tantalum_SMD:CP_EIA-6032-20_AVX-F_Pad2.25x2.35mm_HandSolder, B.Cu at (257.9, 99.1)
- added C501: 1uF, Capacitor_Tantalum_SMD:CP_EIA-6032-20_AVX-F_Pad2.25x2.35mm_HandSolder, B.Cu at (195.5, 99.1)
- added C501: 1uF, Capacitor_Tantalum_SMD:CP_EIA-6032-20_AVX-F_Pad2.25x2.35mm_HandSolder, B.Cu at (133.1, 99.1)
- added C502: 100nF, Capacitor_SMD:C_0805_2012Metric_Pad1.15x1.40mm_HandSolder, B.Cu at (257.9, 95.2)
- added C502: 100nF, Capacitor_SMD:C_0805_2012Metric_Pad1.15x1.40mm_HandSolder, B.Cu at (195.5, 95.2)
- added C502: 100nF, Capacitor_SMD:C_0805_2012Metric_Pad1.15x1.40mm_HandSolder, B.Cu at (133.1, 95.2)
- added C503: 100nF, Capacitor_SMD:C_0805_2012Metric_Pad1.15x1.40mm_HandSolder, B.Cu at (251.3, 98.4)
- added C503: 100nF, Capacitor_SMD:C_0805_2012Metric_Pad1.15x1.40mm_HandSolder, B.Cu at (188.9, 98.4)
- added C503: 100nF, Capacitor_SMD:C_0805_2012Metric_Pad1.15x1.40mm_HandSolder, B.Cu at (126.5, 98.4)
- added C504: 1uF, Capacitor_Tantalum_SMD:CP_EIA-6032-20_AVX-F_Pad2.25x2.35mm_HandSolder, B.Cu at (251.4, 95.2)
- added C504: 1uF, Capacitor_Tantalum_SMD:CP_EIA-6032-20_AVX-F_Pad2.25x2.35mm_HandSolder, B.Cu at (189.0, 95.2)
- added C504: 1uF, Capacitor_Tantalum_SMD:CP_EIA-6032-20_AVX-F_Pad2.25x2.35mm_HandSolder, B.Cu at (126.6, 95.2)
- added D101: LL4148, Diode_SMD:D_MiniMELF_Handsoldering, B.Cu at (228.7, 47.6)
- added D101: LL4148, Diode_SMD:D_MiniMELF_Handsoldering, B.Cu at (166.3, 47.6)
- added D101: LL4148, Diode_SMD:D_MiniMELF_Handsoldering, B.Cu at (103.9, 47.6)
- added D201: pesd1can, Package_TO_SOT_SMD:SOT-23_Handsoldering, B.Cu at (245.9, 128.0)
- added D201: pesd1can, Package_TO_SOT_SMD:SOT-23_Handsoldering, B.Cu at (183.5, 128.0)
- added D201: pesd1can, Package_TO_SOT_SMD:SOT-23_Handsoldering, B.Cu at (121.1, 128.0)
- added D401: LL4148, Diode_SMD:D_MiniMELF_Handsoldering, B.Cu at (224.8, 51.4)
- added D401: LL4148, Diode_SMD:D_MiniMELF_Handsoldering, B.Cu at (162.4, 51.4)
- added D401: LL4148, Diode_SMD:D_MiniMELF_Handsoldering, B.Cu at (100.0, 51.4)
- added D402: LED_RED, LED_SMD:LED_0805_2012Metric_Pad1.15x1.40mm_HandSolder, B.Cu at (224.3, 91.5)
- added D402: LED_RED, LED_SMD:LED_0805_2012Metric_Pad1.15x1.40mm_HandSolder, B.Cu at (161.9, 91.5)
- added D402: LED_RED, LED_SMD:LED_0805_2012Metric_Pad1.15x1.40mm_HandSolder, B.Cu at (99.5, 91.5)
- added D403: LED_RED, LED_SMD:LED_0805_2012Metric_Pad1.15x1.40mm_HandSolder, B.Cu at (224.3, 89.0)
- added D403: LED_RED, LED_SMD:LED_0805_2012Metric_Pad1.15x1.40mm_HandSolder, B.Cu at (161.9, 89.0)
- added D403: LED_RED, LED_SMD:LED_0805_2012Metric_Pad1.15x1.40mm_HandSolder, B.Cu at (99.5, 89.0)
- added D501: LL4148, Diode_SMD:D_MiniMELF_Handsoldering, B.Cu at (263.4, 112.4)
- added D501: LL4148, Diode_SMD:D_MiniMELF_Handsoldering, B.Cu at (201.0, 112.4)
- added D501: LL4148, Diode_SMD:D_MiniMELF_Handsoldering, B.Cu at (138.6, 112.4)
- added F501: 500mA, Fuse:Fuse_1206_3216Metric_Pad1.42x1.75mm_HandSolder, B.Cu at (263.4, 103.5)
- added F501: 500mA, Fuse:Fuse_1206_3216Metric_Pad1.42x1.75mm_HandSolder, B.Cu at (201.0, 103.5)
- added F501: 500mA, Fuse:Fuse_1206_3216Metric_Pad1.42x1.75mm_HandSolder, B.Cu at (138.6, 103.5)
- added H101: MountingHole, MountingHole:MountingHole_3.2mm_M3, F.Cu at (222.1, 40.6)
- added H101: MountingHole, MountingHole:MountingHole_3.2mm_M3, F.Cu at (159.7, 40.6)
- added H101: MountingHole, MountingHole:MountingHole_3.2mm_M3, F.Cu at (97.3, 40.6)
- added H102: MountingHole, MountingHole:MountingHole_3.2mm_M3, F.Cu at (221.7, 126.1)
- added H102: MountingHole, MountingHole:MountingHole_3.2mm_M3, F.Cu at (159.3, 126.1)
- added H102: MountingHole, MountingHole:MountingHole_3.2mm_M3, F.Cu at (96.9, 126.1)
- added H103: MountingHole, MountingHole:MountingHole_3.2mm_M3, F.Cu at (264.0, 125.1)
- added H103: MountingHole, MountingHole:MountingHole_3.2mm_M3, F.Cu at (201.6, 125.1)
- added H103: MountingHole, MountingHole:MountingHole_3.2mm_M3, F.Cu at (139.2, 125.1)
- added H104: MountingHole, MountingHole:MountingHole_3.2mm_M3, F.Cu at (264.0, 40.6)
- added H104: MountingHole, MountingHole:MountingHole_3.2mm_M3, F.Cu at (201.6, 40.6)
- added H104: MountingHole, MountingHole:MountingHole_3.2mm_M3, F.Cu at (139.2, 40.6)
- added J1: Conn_01x04, Connector_PinHeader_2.54mm:PinHeader_1x04_P2.54mm_Vertical, F.Cu at (255.1, 38.7)
- added J1: Conn_01x04, Connector_PinHeader_2.54mm:PinHeader_1x04_P2.54mm_Vertical, F.Cu at (192.7, 38.7)
- added J1: Conn_01x04, Connector_PinHeader_2.54mm:PinHeader_1x04_P2.54mm_Vertical, F.Cu at (130.3, 38.7)
- added J401: USART, Connector_PinHeader_2.54mm:PinHeader_1x04_P2.54mm_Vertical, F.Cu at (221.7, 63.9)
- added J401: USART, Connector_PinHeader_2.54mm:PinHeader_1x04_P2.54mm_Vertical, F.Cu at (159.3, 63.9)
- added J401: USART, Connector_PinHeader_2.54mm:PinHeader_1x04_P2.54mm_Vertical, F.Cu at (96.9, 63.9)
- added J601: RJ45, KicadZeniteSolarLibrary18:RJ45_YH59_01, F.Cu at (248.4, 138.8)
- added J601: RJ45, KicadZeniteSolarLibrary18:RJ45_YH59_01, F.Cu at (186.0, 138.8)
- added J601: RJ45, KicadZeniteSolarLibrary18:RJ45_YH59_01, F.Cu at (123.6, 138.8)
- added J602: RJ45, KicadZeniteSolarLibrary18:RJ45_YH59_01, F.Cu at (227.6, 138.8)
- added J602: RJ45, KicadZeniteSolarLibrary18:RJ45_YH59_01, F.Cu at (165.2, 138.8)
- added J602: RJ45, KicadZeniteSolarLibrary18:RJ45_YH59_01, F.Cu at (102.8, 138.8)
- added R101: 330, Resistor_SMD:R_0805_2012Metric_Pad1.15x1.40mm_HandSolder, B.Cu at (231.3, 44.5)
- added R101: 330, Resistor_SMD:R_0805_2012Metric_Pad1.15x1.40mm_HandSolder, B.Cu at (168.9, 44.5)
- added R101: 330, Resistor_SMD:R_0805_2012Metric_Pad1.15x1.40mm_HandSolder, B.Cu at (106.5, 44.5)
- added R102: 10k, Resistor_SMD:R_0805_2012Metric_Pad1.15x1.40mm_HandSolder, B.Cu at (239.9, 40.0)
- added R102: 10k, Resistor_SMD:R_0805_2012Metric_Pad1.15x1.40mm_HandSolder, B.Cu at (177.5, 40.0)
- added R102: 10k, Resistor_SMD:R_0805_2012Metric_Pad1.15x1.40mm_HandSolder, B.Cu at (115.1, 40.0)
- added R103: 330, Resistor_SMD:R_0805_2012Metric_Pad1.15x1.40mm_HandSolder, B.Cu at (231.3, 41.9)
- added R103: 330, Resistor_SMD:R_0805_2012Metric_Pad1.15x1.40mm_HandSolder, B.Cu at (168.9, 41.9)
- added R103: 330, Resistor_SMD:R_0805_2012Metric_Pad1.15x1.40mm_HandSolder, B.Cu at (106.5, 41.9)
- added R201: 120, Resistor_SMD:R_0805_2012Metric_Pad1.15x1.40mm_HandSolder, B.Cu at (245.9, 124.0)
- added R201: 120, Resistor_SMD:R_0805_2012Metric_Pad1.15x1.40mm_HandSolder, B.Cu at (183.5, 124.0)
- added R201: 120, Resistor_SMD:R_0805_2012Metric_Pad1.15x1.40mm_HandSolder, B.Cu at (121.1, 124.0)
- added R202: 4k7, Resistor_SMD:R_0805_2012Metric_Pad1.15x1.40mm_HandSolder, B.Cu at (237.6, 125.1)
- added R202: 4k7, Resistor_SMD:R_0805_2012Metric_Pad1.15x1.40mm_HandSolder, B.Cu at (175.2, 125.1)
- added R202: 4k7, Resistor_SMD:R_0805_2012Metric_Pad1.15x1.40mm_HandSolder, B.Cu at (112.8, 125.1)
- added R203: 10k, Resistor_SMD:R_0805_2012Metric_Pad1.15x1.40mm_HandSolder, B.Cu at (245.9, 111.1)
- added R203: 10k, Resistor_SMD:R_0805_2012Metric_Pad1.15x1.40mm_HandSolder, B.Cu at (183.5, 111.1)
- added R203: 10k, Resistor_SMD:R_0805_2012Metric_Pad1.15x1.40mm_HandSolder, B.Cu at (121.1, 111.1)
- added R401: 10k, Resistor_SMD:R_0805_2012Metric_Pad1.15x1.40mm_HandSolder, B.Cu at (229.4, 53.7)
- added R401: 10k, Resistor_SMD:R_0805_2012Metric_Pad1.15x1.40mm_HandSolder, B.Cu at (167.0, 53.7)
- added R401: 10k, Resistor_SMD:R_0805_2012Metric_Pad1.15x1.40mm_HandSolder, B.Cu at (104.6, 53.7)
- added R402: 1k, Resistor_SMD:R_0805_2012Metric_Pad1.15x1.40mm_HandSolder, B.Cu at (229.4, 58.8)
- added R402: 1k, Resistor_SMD:R_0805_2012Metric_Pad1.15x1.40mm_HandSolder, B.Cu at (167.0, 58.8)
- added R402: 1k, Resistor_SMD:R_0805_2012Metric_Pad1.15x1.40mm_HandSolder, B.Cu at (104.6, 58.8)
- added R403: 1k, Resistor_SMD:R_0805_2012Metric_Pad1.15x1.40mm_HandSolder, B.Cu at (229.4, 61.3)
- added R403: 1k, Resistor_SMD:R_0805_2012Metric_Pad1.15x1.40mm_HandSolder, B.Cu at (167.0, 61.3)
- added R403: 1k, Resistor_SMD:R_0805_2012Metric_Pad1.15x1.40mm_HandSolder, B.Cu at (104.6, 61.3)
- added R404: 1k, Resistor_SMD:R_0805_2012Metric_Pad1.15x1.40mm_HandSolder, B.Cu at (228.1, 91.5)
- added R404: 1k, Resistor_SMD:R_0805_2012Metric_Pad1.15x1.40mm_HandSolder, B.Cu at (165.7, 91.5)
- added R404: 1k, Resistor_SMD:R_0805_2012Metric_Pad1.15x1.40mm_HandSolder, B.Cu at (103.3, 91.5)
- added R405: 1k, Resistor_SMD:R_0805_2012Metric_Pad1.15x1.40mm_HandSolder, B.Cu at (228.1, 89.0)
- added R405: 1k, Resistor_SMD:R_0805_2012Metric_Pad1.15x1.40mm_HandSolder, B.Cu at (165.7, 89.0)
- added R405: 1k, Resistor_SMD:R_0805_2012Metric_Pad1.15x1.40mm_HandSolder, B.Cu at (103.3, 89.0)
- added R601: 330, Resistor_SMD:R_0805_2012Metric_Pad1.15x1.40mm_HandSolder, B.Cu at (231.4, 39.4)
- added R601: 330, Resistor_SMD:R_0805_2012Metric_Pad1.15x1.40mm_HandSolder, B.Cu at (169.0, 39.4)
- added R601: 330, Resistor_SMD:R_0805_2012Metric_Pad1.15x1.40mm_HandSolder, B.Cu at (106.6, 39.4)
- added TP201: SI, TestPoint:TestPoint_Pad_2.0x2.0mm, B.Cu at (249.4, 104.8)
- added TP201: SI, TestPoint:TestPoint_Pad_2.0x2.0mm, B.Cu at (187.0, 104.8)
- added TP201: SI, TestPoint:TestPoint_Pad_2.0x2.0mm, B.Cu at (124.6, 104.8)
- added TP202: SO, TestPoint:TestPoint_Pad_2.0x2.0mm, B.Cu at (249.4, 108.0)
- added TP202: SO, TestPoint:TestPoint_Pad_2.0x2.0mm, B.Cu at (187.0, 108.0)
- added TP202: SO, TestPoint:TestPoint_Pad_2.0x2.0mm, B.Cu at (124.6, 108.0)
- added TP203: TXCAN, TestPoint:TestPoint_Pad_2.0x2.0mm, B.Cu at (227.2, 115.6)
- added TP203: TXCAN, TestPoint:TestPoint_Pad_2.0x2.0mm, B.Cu at (164.8, 115.6)
- added TP203: TXCAN, TestPoint:TestPoint_Pad_2.0x2.0mm, B.Cu at (102.4, 115.6)
- added TP204: RXCAN, TestPoint:TestPoint_Pad_2.0x2.0mm, B.Cu at (227.2, 111.1)
- added TP204: RXCAN, TestPoint:TestPoint_Pad_2.0x2.0mm, B.Cu at (164.8, 111.1)
- added TP204: RXCAN, TestPoint:TestPoint_Pad_2.0x2.0mm, B.Cu at (102.4, 111.1)
- added TP205: SC, TestPoint:TestPoint_Pad_2.0x2.0mm, B.Cu at (249.4, 111.1)
- added TP205: SC, TestPoint:TestPoint_Pad_2.0x2.0mm, B.Cu at (187.0, 111.1)
- added TP205: SC, TestPoint:TestPoint_Pad_2.0x2.0mm, B.Cu at (124.6, 111.1)
- added TP206: SCK, TestPoint:TestPoint_Pad_2.0x2.0mm, B.Cu at (249.4, 101.6)
- added TP206: SCK, TestPoint:TestPoint_Pad_2.0x2.0mm, B.Cu at (187.0, 101.6)
- added TP206: SCK, TestPoint:TestPoint_Pad_2.0x2.0mm, B.Cu at (124.6, 101.6)
- added TP207: CAN_H, TestPoint:TestPoint_Pad_2.0x2.0mm, B.Cu at (242.4, 123.8)
- added TP207: CAN_H, TestPoint:TestPoint_Pad_2.0x2.0mm, B.Cu at (180.0, 123.8)
- added TP207: CAN_H, TestPoint:TestPoint_Pad_2.0x2.0mm, B.Cu at (117.6, 123.8)
- added TP208: CAN_L, TestPoint:TestPoint_Pad_2.0x2.0mm, B.Cu at (249.4, 123.8)
- added TP208: CAN_L, TestPoint:TestPoint_Pad_2.0x2.0mm, B.Cu at (187.0, 123.8)
- added TP208: CAN_L, TestPoint:TestPoint_Pad_2.0x2.0mm, B.Cu at (124.6, 123.8)
- added TP209: INT, TestPoint:TestPoint_Pad_2.0x2.0mm, B.Cu at (243.1, 92.1)
- added TP209: INT, TestPoint:TestPoint_Pad_2.0x2.0mm, B.Cu at (180.7, 92.1)
- added TP209: INT, TestPoint:TestPoint_Pad_2.0x2.0mm, B.Cu at (118.3, 92.1)
- added U201: MCP2551-I/SN, Package_SO:SOIC-8_3.9x4.9mm_P1.27mm, B.Cu at (237.6, 117.9)
- added U201: MCP2551-I/SN, Package_SO:SOIC-8_3.9x4.9mm_P1.27mm, B.Cu at (175.2, 117.9)
- added U201: MCP2551-I/SN, Package_SO:SOIC-8_3.9x4.9mm_P1.27mm, B.Cu at (112.8, 117.9)
- added U202: MCP2515-xSO, Package_SO:SOIC-18W_7.5x11.6mm_P1.27mm, B.Cu at (237.6, 105.8)
- added U202: MCP2515-xSO, Package_SO:SOIC-18W_7.5x11.6mm_P1.27mm, B.Cu at (175.2, 105.8)
- added U202: MCP2515-xSO, Package_SO:SOIC-18W_7.5x11.6mm_P1.27mm, B.Cu at (112.8, 105.8)
- added U301: A1101ELHL, Package_TO_SOT_SMD:SOT-23, B.Cu at (239.9, 43.5)
- added U301: A1101ELHL, Package_TO_SOT_SMD:SOT-23, B.Cu at (177.5, 43.5)
- added U301: A1101ELHL, Package_TO_SOT_SMD:SOT-23, B.Cu at (115.1, 43.5)
- added U401: ATMEGA328P-PU, Package_DIP:DIP-28_W7.62mm_Socket, F.Cu at (234.4, 56.3)
- added U401: ATMEGA328P-PU, Package_DIP:DIP-28_W7.62mm_Socket, F.Cu at (172.0, 56.3)
- added U401: ATMEGA328P-PU, Package_DIP:DIP-28_W7.62mm_Socket, F.Cu at (109.6, 56.3)
- added U501: LM7805, KicadZeniteSolarLibrary18:TO-220-3_Horizontal_TabDown_SMD, B.Cu at (257.1, 89.5)
- added U501: LM7805, KicadZeniteSolarLibrary18:TO-220-3_Horizontal_TabDown_SMD, B.Cu at (194.7, 89.5)
- added U501: LM7805, KicadZeniteSolarLibrary18:TO-220-3_Horizontal_TabDown_SMD, B.Cu at (132.2, 89.5)
- added Y201: 16MHz, Crystal:Crystal_HC49-U_Vertical, F.Cu at (226.8, 105.8)
- added Y201: 16MHz, Crystal:Crystal_HC49-U_Vertical, F.Cu at (164.4, 105.8)
- added Y201: 16MHz, Crystal:Crystal_HC49-U_Vertical, F.Cu at (102.0, 105.8)
- added Y401: 16MHz, Crystal:Crystal_HC49-U_Vertical, F.Cu at (228.1, 81.7)
- added Y401: 16MHz, Crystal:Crystal_HC49-U_Vertical, F.Cu at (165.7, 81.7)
- added Y401: 16MHz, Crystal:Crystal_HC49-U_Vertical, F.Cu at (103.3, 81.7)
- added Z101: 4.7V, Diode_SMD:D_MiniMELF_Handsoldering, B.Cu at (235.5, 45.9)
- added Z101: 4.7V, Diode_SMD:D_MiniMELF_Handsoldering, B.Cu at (173.1, 45.9)
- added Z101: 4.7V, Diode_SMD:D_MiniMELF_Handsoldering, B.Cu at (110.7, 45.9)
- added Z102: 4.7V, Diode_SMD:D_MiniMELF_Handsoldering, B.Cu at (242.7, 47.6)
- added Z102: 4.7V, Diode_SMD:D_MiniMELF_Handsoldering, B.Cu at (180.3, 47.6)
- added Z102: 4.7V, Diode_SMD:D_MiniMELF_Handsoldering, B.Cu at (117.9, 47.6)
- moved C1 31.0 mm to (51.8, 50.8)
- moved C101 31.0 mm to (48.0, 39.4)
- moved C201 31.0 mm to (47.6, 97.2)
- moved C204 31.0 mm to (42.2, 99.4)
- moved C205 31.0 mm to (50.4, 122.9)
- moved C402 31.0 mm to (43.4, 71.5)
- moved C404 31.0 mm to (42.2, 74.7)
- moved C405 31.0 mm to (42.2, 56.3)
- moved C406 31.0 mm to (44.6, 51.3)
- moved C501 31.0 mm to (70.7, 99.1)
- moved C504 31.0 mm to (64.2, 95.2)
- moved D101 31.0 mm to (41.5, 47.6)
- moved D501 31.0 mm to (76.2, 112.4)
- moved F501 31.0 mm to (76.2, 103.5)
- moved H101 31.0 mm to (34.9, 40.6)
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Routing:
- net +5V: track 209.3 -> 837.0 mm
- net GND: track 97.6 -> 390.2 mm, vias 16 -> 64
- net /POWER SUPPLY/+18V_IN: track 71.9 -> 287.8 mm
- net /CANBUS CONN/CAN_H: track 53.1 -> 212.5 mm
- net /CANBUS CONN/CAN_L: track 51.4 -> 205.5 mm, vias 2 -> 8
- net /MISO: track 37.7 -> 150.9 mm
- net /MCU/VOUT: track 36.4 -> 145.6 mm
- net /SCK: track 35.6 -> 142.3 mm
- net /MOSI: track 32.9 -> 131.5 mm
- net /CANBUS/CS: track 32.2 -> 128.6 mm
- net /MCU/SDA: track 25.7 -> 103.0 mm
- net /MCU/SCL: track 22.5 -> 90.1 mm
- net /CANBUS/INT: track 21.3 -> 85.0 mm
- net Net-(C101-Pad1): track 16.9 -> 67.7 mm
- net /CANBUS/TXCAN: track 16.5 -> 65.8 mm
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Other:
- board size 52.1 x 121.3 mm -> 239.3 x 121.3 mm
