File: hardware/basicsensormodule.kicad_pcb (KiCad board)
At the start: 2 copper layers, 247.1 x 121 mm, 212 parts, among them J1 Conn_01x04, J401 USART, J601 RJ45, J602 RJ45, U201 MCP2551-I/SN, U202 MCP2515-xSO, U401 ATMEGA328P-PU, U501 LM7805, Y201 16MHz, Y401 16MHz

Commit message: Layout MT19 criado para o Taquímetro do barco.
Parts:
- removed the C102 at (237.5, 43.4)
- removed the C102 at (172.5, 43.4)
- removed the C102 at (107.5, 43.4)
- removed the C201 at (235.0, 94.0)
- removed the C201 at (170.0, 94.0)
- removed the C201 at (105.0, 94.0)
- removed the C202 at (242.6, 109.9)
- removed the C202 at (177.6, 109.9)
- removed the C202 at (112.6, 109.9)
- removed the C203 at (227.4, 100.1)
- removed the C203 at (162.4, 100.1)
- removed the C203 at (97.4, 100.1)
- removed the C204 at (229.5, 96.3)
- removed the C204 at (164.5, 96.3)
- removed the C204 at (99.5, 96.3)
- removed the C205 at (237.8, 119.8)
- removed the C205 at (172.8, 119.8)
- removed the C205 at (107.8, 119.8)
- removed the C401 at (246.1, 73.4)
- removed the C401 at (181.1, 73.4)
- removed the C401 at (116.1, 73.4)
- removed the C402 at (230.8, 68.3)
- removed the C402 at (165.8, 68.3)
- removed the C402 at (100.8, 68.3)
- removed the C403 at (228.3, 75.9)
- removed the C403 at (163.3, 75.9)
- removed the C403 at (98.3, 75.9)
- removed the C404 at (229.5, 71.5)
- removed the C404 at (164.5, 71.5)
- removed the C404 at (99.5, 71.5)
- removed the C405 at (229.5, 53.1)
- removed the C405 at (164.5, 53.1)
- removed the C405 at (99.5, 53.1)
- removed the C406 at (232.0, 48.1)
- removed the C406 at (167.0, 48.1)
- removed the C406 at (102.0, 48.1)
- removed the C501 at (258.1, 95.9)
- removed the C501 at (193.1, 95.9)
- removed the C501 at (128.1, 95.9)
- removed the C502 at (258.1, 92.1)
- removed the C502 at (193.1, 92.1)
- removed the C502 at (128.1, 92.1)
- removed the C503 at (251.5, 95.2)
- removed the C503 at (186.5, 95.2)
- removed the C503 at (121.5, 95.2)
- removed the C504 at (251.5, 92.1)
- removed the C504 at (186.5, 92.1)
- removed the C504 at (121.5, 92.1)
- removed the D201 at (246.1, 124.8)
- removed the D201 at (181.1, 124.8)
- removed the D201 at (116.1, 124.8)
- removed the D401 at (225.0, 48.3)
- removed the D401 at (160.0, 48.3)
- removed the D401 at (95.0, 48.3)
- removed the D402 at (224.5, 88.4)
- removed the D402 at (159.5, 88.4)
- removed the D402 at (94.5, 88.4)
- removed the D403 at (224.5, 85.8)
- removed the D403 at (159.5, 85.8)
- removed the D403 at (94.5, 85.8)
- removed the D501 at (263.6, 109.2)
- removed the D501 at (198.6, 109.2)
- removed the D501 at (133.6, 109.2)
- removed the F501 at (263.6, 100.3)
- removed the F501 at (198.6, 100.3)
- removed the F501 at (133.6, 100.3)
- removed the H101 at (222.9, 38.1)
- removed the H101 at (157.9, 38.1)
- removed the H101 at (92.9, 38.1)
- removed the H102 at (221.9, 122.9)
- removed the H102 at (156.9, 122.9)
- removed the H102 at (91.9, 122.9)
- removed the H103 at (265.1, 122.9)
- removed the H103 at (200.1, 122.9)
- removed the H103 at (135.1, 122.9)
- removed the H104 at (264.9, 38.1)
- removed the H104 at (199.8, 38.1)
- removed the H104 at (134.8, 38.1)
- removed the J1 at (244.5, 38.1)
- removed the J1 at (179.5, 38.1)
- removed the J1 at (114.5, 38.1)
- removed the J401 at (221.9, 60.7)
- removed the J401 at (156.9, 60.7)
- removed the J401 at (91.9, 60.7)
- removed the J601 at (248.6, 135.6)
- removed the J601 at (183.6, 135.6)
- removed the J601 at (118.6, 135.6)
- removed the J602 at (227.7, 135.6)
- removed the J602 at (162.7, 135.6)
- removed the J602 at (97.7, 135.6)
- removed the R201 at (246.1, 120.8)
- removed the R201 at (181.1, 120.8)
- removed the R201 at (116.1, 120.8)
- removed the R202 at (237.8, 121.9)
- removed the R202 at (172.8, 121.9)
- removed the R202 at (107.8, 121.9)
- removed the R203 at (246.0, 108.0)
- removed the R203 at (181.0, 108.0)
- removed the R203 at (116.0, 108.0)
- removed the R401 at (229.5, 50.5)
- removed the R401 at (164.5, 50.5)
- removed the R401 at (99.5, 50.5)
- removed the R402 at (229.5, 55.6)
- removed the R402 at (164.5, 55.6)
- removed the R402 at (99.5, 55.6)
- removed the R403 at (229.5, 58.2)
- removed the R403 at (164.5, 58.2)
- removed the R403 at (99.5, 58.2)
- removed the R404 at (228.3, 88.4)
- removed the R404 at (163.3, 88.4)
- removed the R404 at (98.3, 88.4)
- removed the R405 at (228.3, 85.8)
- removed the R405 at (163.3, 85.8)
- removed the R405 at (98.3, 85.8)
- removed the TP201 at (250.0, 101.6)
- removed the TP201 at (185.0, 101.6)
- removed the TP201 at (120.0, 101.6)
- removed the TP202 at (250.0, 104.8)
- removed the TP202 at (185.0, 104.8)
- removed the TP202 at (120.0, 104.8)
- removed the TP203 at (228.9, 112.1)
- removed the TP203 at (163.9, 112.1)
- removed the TP203 at (98.9, 112.1)
- removed the TP204 at (228.9, 108.3)
- removed the TP204 at (163.9, 108.3)
- removed the TP204 at (98.9, 108.3)
- removed the TP205 at (250.0, 108.0)
- removed the TP205 at (185.0, 108.0)
- removed the TP205 at (120.0, 108.0)
- removed the TP206 at (250.0, 98.4)
- removed the TP206 at (185.0, 98.4)
- removed the TP206 at (120.0, 98.4)
- removed the TP207 at (244.1, 118.1)
- removed the TP207 at (179.1, 118.1)
- removed the TP207 at (114.1, 118.1)
- removed the TP208 at (246.7, 114.7)
- removed the TP208 at (181.7, 114.7)
- removed the TP208 at (116.7, 114.7)
- removed the TP209 at (243.3, 89.2)
- removed the TP209 at (178.3, 89.2)
- removed the TP209 at (113.3, 89.2)
- removed the U201 at (237.8, 114.7)
- removed the U201 at (172.8, 114.7)
- removed the U201 at (107.8, 114.7)
- removed the U202 at (237.8, 102.6)
- removed the U202 at (172.8, 102.6)
- removed the U202 at (107.8, 102.6)
- removed the U401 at (234.6, 53.1)
- removed the U401 at (169.6, 53.1)
- removed the U401 at (104.6, 53.1)
- removed the U501 at (257.2, 86.4)
- removed the U501 at (192.2, 86.4)
- removed the U501 at (127.2, 86.4)
- removed the Y201 at (227.0, 102.6)
- removed the Y201 at (162.0, 102.6)
- removed the Y201 at (97.0, 102.6)
- removed the Y401 at (228.3, 78.5)
- removed the Y401 at (163.3, 78.5)
- removed the Y401 at (98.3, 78.5)
- added C1: 4.7n, Capacitor_SMD:C_0805_2012Metric_Pad1.15x1.40mm_HandSolder, B.Cu at (82.3, 56.5)
- added C101: 100n, Capacitor_SMD:C_0805_2012Metric_Pad1.15x1.40mm_HandSolder, B.Cu at (74.7, 48.3)
- added D101: LL4148, Diode_SMD:D_MiniMELF_Handsoldering, B.Cu at (72.0, 53.3)
- added R101: 100, Resistor_SMD:R_0805_2012Metric_Pad1.15x1.40mm_HandSolder, B.Cu at (74.7, 50.8)
- added U301: A1101ELHL, Package_TO_SOT_SMD:SOT-23, B.Cu at (83.2, 49.3)
- added Z101: 4.7V, Diode_SMD:D_MiniMELF_Handsoldering, B.Cu at (78.7, 51.6)
- added Z102: 4.7V, Diode_SMD:D_MiniMELF_Handsoldering, B.Cu at (85.9, 53.3)
- moved J1 49.5 mm to (98.4, 45.7)
- moved C204 39.1 mm to (72.6, 105.2)
- moved C404 39.1 mm to (72.6, 80.4)
- moved C405 39.1 mm to (72.6, 62.0)
- moved D501 39.1 mm to (106.7, 118.1)
- moved F501 39.1 mm to (106.7, 109.2)
- moved R401 39.1 mm to (72.6, 59.4)
- moved R402 39.1 mm to (72.6, 64.5)
- moved R403 39.1 mm to (72.6, 67.1)
- moved C201 39.1 mm to (78.1, 102.9)
- moved C203 39.1 mm to (70.5, 109.0)
- moved C205 39.1 mm to (80.9, 128.7)
- moved C402 39.1 mm to (73.9, 77.2)
- moved C406 39.1 mm to (75.1, 57.0)
- moved C501 39.1 mm to (101.2, 104.8)
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Connections:
- U401 pad 4: Net-(U401-Pad4) -> /MCU/VOUT
- U501 pad : GND -> (no net)
Routing:
- net +5V: track 807.1 -> 202.9 mm
- net GND: track 318.1 -> 82.6 mm, vias 56 -> 14
- net /POWER SUPPLY/+18V_IN: track 287.8 -> 71.9 mm
- net /CANBUS CONN/CAN_H: track 202.3 -> 50.6 mm
- net /CANBUS CONN/CAN_L: track 192.7 -> 48.2 mm, vias 8 -> 2
- net /MISO: track 150.9 -> 37.7 mm
- net /SCK: track 142.3 -> 35.6 mm
- net /MOSI: track 131.5 -> 32.9 mm
- net /CANBUS/CS: track 128.6 -> 32.2 mm
- net /MCU/SDA: track 92.5 -> 25.2 mm
- net /CANBUS/INT: track 84.4 -> 21.1 mm
- net /CANBUS/TXCAN: track 61.4 -> 15.4 mm
- net /CANBUS/RXCAN: track 56.5 -> 14.1 mm
- net /POWER SUPPLY/+18V_OUT: track 55.4 -> 13.8 mm
- net /MCU/SCL: track 60.4 -> 22.0 mm
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Other:
- board size 247.1 x 121 mm -> 52.1 x 121.3 mm

Commit message: layout finalizado
Parts:
- removed the C101 at (74.7, 48.3)
- removed the C102 at (73.7, 44.5)
- removed the TP201 at (93.1, 110.5)
- removed the TP202 at (93.1, 113.7)
- removed the TP203 at (72.0, 121.0)
- removed the TP204 at (72.0, 117.2)
- removed the TP205 at (93.1, 116.8)
- removed the TP206 at (93.1, 107.3)
- removed the TP207 at (87.2, 127.0)
- removed the TP208 at (89.8, 123.6)
- removed the TP209 at (86.4, 98.0)
- added C1: 4.7n, Capacitor_SMD:C_0805_2012Metric_Pad1.15x1.40mm_HandSolder, B.Cu at (239.0, 50.8)
- added C1: 4.7n, Capacitor_SMD:C_0805_2012Metric_Pad1.15x1.40mm_HandSolder, B.Cu at (176.6, 50.8)
- added C1: 4.7n, Capacitor_SMD:C_0805_2012Metric_Pad1.15x1.40mm_HandSolder, B.Cu at (114.2, 50.8)
- added C101: 100n, Capacitor_SMD:C_0805_2012Metric_Pad1.15x1.40mm_HandSolder, B.Cu at (235.2, 39.4)
- added C101: 100n, Capacitor_SMD:C_0805_2012Metric_Pad1.15x1.40mm_HandSolder, B.Cu at (172.8, 39.4)
- added C101: 100n, Capacitor_SMD:C_0805_2012Metric_Pad1.15x1.40mm_HandSolder, B.Cu at (110.4, 39.4)
- added C101: 100n, Capacitor_SMD:C_0805_2012Metric_Pad1.15x1.40mm_HandSolder, B.Cu at (48.0, 39.4)
- added C102: 100nF, Capacitor_SMD:C_0805_2012Metric_Pad1.15x1.40mm_HandSolder, B.Cu at (248.6, 41.9)
- added C102: 100nF, Capacitor_SMD:C_0805_2012Metric_Pad1.15x1.40mm_HandSolder, B.Cu at (186.2, 41.9)
- added C102: 100nF, Capacitor_SMD:C_0805_2012Metric_Pad1.15x1.40mm_HandSolder, B.Cu at (123.8, 41.9)
- added C102: 100nF, Capacitor_SMD:C_0805_2012Metric_Pad1.15x1.40mm_HandSolder, B.Cu at (61.4, 41.9)
- added C201: 100nF, Capacitor_SMD:C_0805_2012Metric_Pad1.15x1.40mm_HandSolder, B.Cu at (234.8, 97.2)
- added C201: 100nF, Capacitor_SMD:C_0805_2012Metric_Pad1.15x1.40mm_HandSolder, B.Cu at (172.4, 97.2)
- added C201: 100nF, Capacitor_SMD:C_0805_2012Metric_Pad1.15x1.40mm_HandSolder, B.Cu at (110.0, 97.2)
- added C202: 100nF, Capacitor_SMD:C_0805_2012Metric_Pad1.15x1.40mm_HandSolder, B.Cu at (242.4, 113.0)
- added C202: 100nF, Capacitor_SMD:C_0805_2012Metric_Pad1.15x1.40mm_HandSolder, B.Cu at (180.0, 113.0)
- added C202: 100nF, Capacitor_SMD:C_0805_2012Metric_Pad1.15x1.40mm_HandSolder, B.Cu at (117.6, 113.0)
- added C203: 22pF, Capacitor_SMD:C_0805_2012Metric_Pad1.15x1.40mm_HandSolder, B.Cu at (227.2, 103.3)
- added C203: 22pF, Capacitor_SMD:C_0805_2012Metric_Pad1.15x1.40mm_HandSolder, B.Cu at (164.8, 103.3)
- added C203: 22pF, Capacitor_SMD:C_0805_2012Metric_Pad1.15x1.40mm_HandSolder, B.Cu at (102.4, 103.3)
- added C204: 22pF, Capacitor_SMD:C_0805_2012Metric_Pad1.15x1.40mm_HandSolder, B.Cu at (229.4, 99.4)
- added C204: 22pF, Capacitor_SMD:C_0805_2012Metric_Pad1.15x1.40mm_HandSolder, B.Cu at (167.0, 99.4)
- added C204: 22pF, Capacitor_SMD:C_0805_2012Metric_Pad1.15x1.40mm_HandSolder, B.Cu at (104.6, 99.4)
- added C205: 100nF, Capacitor_SMD:C_0805_2012Metric_Pad1.15x1.40mm_HandSolder, B.Cu at (237.6, 122.9)
- added C205: 100nF, Capacitor_SMD:C_0805_2012Metric_Pad1.15x1.40mm_HandSolder, B.Cu at (175.2, 122.9)
- added C205: 100nF, Capacitor_SMD:C_0805_2012Metric_Pad1.15x1.40mm_HandSolder, B.Cu at (112.8, 122.9)
- added C401: 100nF, Capacitor_SMD:C_0805_2012Metric_Pad1.15x1.40mm_HandSolder, B.Cu at (245.9, 76.6)
- added C401: 100nF, Capacitor_SMD:C_0805_2012Metric_Pad1.15x1.40mm_HandSolder, B.Cu at (183.5, 76.6)
- added C401: 100nF, Capacitor_SMD:C_0805_2012Metric_Pad1.15x1.40mm_HandSolder, B.Cu at (121.1, 76.6)
- added C402: 100nF, Capacitor_SMD:C_0805_2012Metric_Pad1.15x1.40mm_HandSolder, B.Cu at (230.6, 71.5)
- added C402: 100nF, Capacitor_SMD:C_0805_2012Metric_Pad1.15x1.40mm_HandSolder, B.Cu at (168.2, 71.5)
- added C402: 100nF, Capacitor_SMD:C_0805_2012Metric_Pad1.15x1.40mm_HandSolder, B.Cu at (105.8, 71.5)
- added C403: 22pF, Capacitor_SMD:C_0805_2012Metric_Pad1.15x1.40mm_HandSolder, B.Cu at (228.1, 79.1)
- added C403: 22pF, Capacitor_SMD:C_0805_2012Metric_Pad1.15x1.40mm_HandSolder, B.Cu at (165.7, 79.1)
- added C403: 22pF, Capacitor_SMD:C_0805_2012Metric_Pad1.15x1.40mm_HandSolder, B.Cu at (103.3, 79.1)
- added C404: 22pF, Capacitor_SMD:C_0805_2012Metric_Pad1.15x1.40mm_HandSolder, B.Cu at (229.4, 74.7)
- added C404: 22pF, Capacitor_SMD:C_0805_2012Metric_Pad1.15x1.40mm_HandSolder, B.Cu at (167.0, 74.7)
- added C404: 22pF, Capacitor_SMD:C_0805_2012Metric_Pad1.15x1.40mm_HandSolder, B.Cu at (104.6, 74.7)
- added C405: 100nF, Capacitor_SMD:C_0805_2012Metric_Pad1.15x1.40mm_HandSolder, B.Cu at (229.4, 56.3)
- added C405: 100nF, Capacitor_SMD:C_0805_2012Metric_Pad1.15x1.40mm_HandSolder, B.Cu at (167.0, 56.3)
- added C405: 100nF, Capacitor_SMD:C_0805_2012Metric_Pad1.15x1.40mm_HandSolder, B.Cu at (104.6, 56.3)
- added C406: 100nF, Capacitor_SMD:C_0805_2012Metric_Pad1.15x1.40mm_HandSolder, B.Cu at (231.8, 51.3)
- added C406: 100nF, Capacitor_SMD:C_0805_2012Metric_Pad1.15x1.40mm_HandSolder, B.Cu at (169.4, 51.3)
- added C406: 100nF, Capacitor_SMD:C_0805_2012Metric_Pad1.15x1.40mm_HandSolder, B.Cu at (107.0, 51.3)
- added C501: 1uF, Capacitor_Tantalum_SMD:CP_EIA-6032-20_AVX-F_Pad2.25x2.35mm_HandSolder, B.Cu at (257.9, 99.1)
- added C501: 1uF, Capacitor_Tantalum_SMD:CP_EIA-6032-20_AVX-F_Pad2.25x2.35mm_HandSolder, B.Cu at (195.5, 99.1)
- added C501: 1uF, Capacitor_Tantalum_SMD:CP_EIA-6032-20_AVX-F_Pad2.25x2.35mm_HandSolder, B.Cu at (133.1, 99.1)
- added C502: 100nF, Capacitor_SMD:C_0805_2012Metric_Pad1.15x1.40mm_HandSolder, B.Cu at (257.9, 95.2)
- added C502: 100nF, Capacitor_SMD:C_0805_2012Metric_Pad1.15x1.40mm_HandSolder, B.Cu at (195.5, 95.2)
- added C502: 100nF, Capacitor_SMD:C_0805_2012Metric_Pad1.15x1.40mm_HandSolder, B.Cu at (133.1, 95.2)
- added C503: 100nF, Capacitor_SMD:C_0805_2012Metric_Pad1.15x1.40mm_HandSolder, B.Cu at (251.3, 98.4)
- added C503: 100nF, Capacitor_SMD:C_0805_2012Metric_Pad1.15x1.40mm_HandSolder, B.Cu at (188.9, 98.4)
- added C503: 100nF, Capacitor_SMD:C_0805_2012Metric_Pad1.15x1.40mm_HandSolder, B.Cu at (126.5, 98.4)
- added C504: 1uF, Capacitor_Tantalum_SMD:CP_EIA-6032-20_AVX-F_Pad2.25x2.35mm_HandSolder, B.Cu at (251.4, 95.2)
- added C504: 1uF, Capacitor_Tantalum_SMD:CP_EIA-6032-20_AVX-F_Pad2.25x2.35mm_HandSolder, B.Cu at (189.0, 95.2)
- added C504: 1uF, Capacitor_Tantalum_SMD:CP_EIA-6032-20_AVX-F_Pad2.25x2.35mm_HandSolder, B.Cu at (126.6, 95.2)
- added D101: LL4148, Diode_SMD:D_MiniMELF_Handsoldering, B.Cu at (228.7, 47.6)
- added D101: LL4148, Diode_SMD:D_MiniMELF_Handsoldering, B.Cu at (166.3, 47.6)
- added D101: LL4148, Diode_SMD:D_MiniMELF_Handsoldering, B.Cu at (103.9, 47.6)
- added D201: pesd1can, Package_TO_SOT_SMD:SOT-23_Handsoldering, B.Cu at (245.9, 128.0)
- added D201: pesd1can, Package_TO_SOT_SMD:SOT-23_Handsoldering, B.Cu at (183.5, 128.0)
- added D201: pesd1can, Package_TO_SOT_SMD:SOT-23_Handsoldering, B.Cu at (121.1, 128.0)
- added D401: LL4148, Diode_SMD:D_MiniMELF_Handsoldering, B.Cu at (224.8, 51.4)
- added D401: LL4148, Diode_SMD:D_MiniMELF_Handsoldering, B.Cu at (162.4, 51.4)
- added D401: LL4148, Diode_SMD:D_MiniMELF_Handsoldering, B.Cu at (100.0, 51.4)
- added D402: LED_RED, LED_SMD:LED_0805_2012Metric_Pad1.15x1.40mm_HandSolder, B.Cu at (224.3, 91.5)
- added D402: LED_RED, LED_SMD:LED_0805_2012Metric_Pad1.15x1.40mm_HandSolder, B.Cu at (161.9, 91.5)
- added D402: LED_RED, LED_SMD:LED_0805_2012Metric_Pad1.15x1.40mm_HandSolder, B.Cu at (99.5, 91.5)
- added D403: LED_RED, LED_SMD:LED_0805_2012Metric_Pad1.15x1.40mm_HandSolder, B.Cu at (224.3, 89.0)
- added D403: LED_RED, LED_SMD:LED_0805_2012Metric_Pad1.15x1.40mm_HandSolder, B.Cu at (161.9, 89.0)
- added D403: LED_RED, LED_SMD:LED_0805_2012Metric_Pad1.15x1.40mm_HandSolder, B.Cu at (99.5, 89.0)
- added D501: LL4148, Diode_SMD:D_MiniMELF_Handsoldering, B.Cu at (263.4, 112.4)
- added D501: LL4148, Diode_SMD:D_MiniMELF_Handsoldering, B.Cu at (201.0, 112.4)
- added D501: LL4148, Diode_SMD:D_MiniMELF_Handsoldering, B.Cu at (138.6, 112.4)
- added F501: 500mA, Fuse:Fuse_1206_3216Metric_Pad1.42x1.75mm_HandSolder, B.Cu at (263.4, 103.5)
- added F501: 500mA, Fuse:Fuse_1206_3216Metric_Pad1.42x1.75mm_HandSolder, B.Cu at (201.0, 103.5)
- added F501: 500mA, Fuse:Fuse_1206_3216Metric_Pad1.42x1.75mm_HandSolder, B.Cu at (138.6, 103.5)
- added H101: MountingHole, MountingHole:MountingHole_3.2mm_M3, F.Cu at (222.1, 40.6)
- added H101: MountingHole, MountingHole:MountingHole_3.2mm_M3, F.Cu at (159.7, 40.6)
- added H101: MountingHole, MountingHole:MountingHole_3.2mm_M3, F.Cu at (97.3, 40.6)
- added H102: MountingHole, MountingHole:MountingHole_3.2mm_M3, F.Cu at (221.7, 126.1)
- added H102: MountingHole, MountingHole:MountingHole_3.2mm_M3, F.Cu at (159.3, 126.1)
- added H102: MountingHole, MountingHole:MountingHole_3.2mm_M3, F.Cu at (96.9, 126.1)
- added H103: MountingHole, MountingHole:MountingHole_3.2mm_M3, F.Cu at (264.0, 125.1)
- added H103: MountingHole, MountingHole:MountingHole_3.2mm_M3, F.Cu at (201.6, 125.1)
- added H103: MountingHole, MountingHole:MountingHole_3.2mm_M3, F.Cu at (139.2, 125.1)
- added H104: MountingHole, MountingHole:MountingHole_3.2mm_M3, F.Cu at (264.0, 40.6)
- added H104: MountingHole, MountingHole:MountingHole_3.2mm_M3, F.Cu at (201.6, 40.6)
- added H104: MountingHole, MountingHole:MountingHole_3.2mm_M3, F.Cu at (139.2, 40.6)
- added J1: Conn_01x04, Connector_PinHeader_2.54mm:PinHeader_1x04_P2.54mm_Vertical, F.Cu at (255.1, 38.7)
- added J1: Conn_01x04, Connector_PinHeader_2.54mm:PinHeader_1x04_P2.54mm_Vertical, F.Cu at (192.7, 38.7)
- added J1: Conn_01x04, Connector_PinHeader_2.54mm:PinHeader_1x04_P2.54mm_Vertical, F.Cu at (130.3, 38.7)
- added J401: USART, Connector_PinHeader_2.54mm:PinHeader_1x04_P2.54mm_Vertical, F.Cu at (221.7, 63.9)
- added J401: USART, Connector_PinHeader_2.54mm:PinHeader_1x04_P2.54mm_Vertical, F.Cu at (159.3, 63.9)
- added J401: USART, Connector_PinHeader_2.54mm:PinHeader_1x04_P2.54mm_Vertical, F.Cu at (96.9, 63.9)
- added J601: RJ45, KicadZeniteSolarLibrary18:RJ45_YH59_01, F.Cu at (248.4, 138.8)
- added J601: RJ45, KicadZeniteSolarLibrary18:RJ45_YH59_01, F.Cu at (186.0, 138.8)
- added J601: RJ45, KicadZeniteSolarLibrary18:RJ45_YH59_01, F.Cu at (123.6, 138.8)
- added J602: RJ45, KicadZeniteSolarLibrary18:RJ45_YH59_01, F.Cu at (227.6, 138.8)
- added J602: RJ45, KicadZeniteSolarLibrary18:RJ45_YH59_01, F.Cu at (165.2, 138.8)
- added J602: RJ45, KicadZeniteSolarLibrary18:RJ45_YH59_01, F.Cu at (102.8, 138.8)
- added R101: 330, Resistor_SMD:R_0805_2012Metric_Pad1.15x1.40mm_HandSolder, B.Cu at (231.3, 44.5)
- added R101: 330, Resistor_SMD:R_0805_2012Metric_Pad1.15x1.40mm_HandSolder, B.Cu at (168.9, 44.5)
- added R101: 330, Resistor_SMD:R_0805_2012Metric_Pad1.15x1.40mm_HandSolder, B.Cu at (106.5, 44.5)
- added R102: 10k, Resistor_SMD:R_0805_2012Metric_Pad1.15x1.40mm_HandSolder, B.Cu at (239.9, 40.0)
- added R102: 10k, Resistor_SMD:R_0805_2012Metric_Pad1.15x1.40mm_HandSolder, B.Cu at (177.5, 40.0)
- added R102: 10k, Resistor_SMD:R_0805_2012Metric_Pad1.15x1.40mm_HandSolder, B.Cu at (115.1, 40.0)
- added R102: 10k, Resistor_SMD:R_0805_2012Metric_Pad1.15x1.40mm_HandSolder, B.Cu at (52.7, 40.0)
- added R103: 330, Resistor_SMD:R_0805_2012Metric_Pad1.15x1.40mm_HandSolder, B.Cu at (231.3, 41.9)
- added R103: 330, Resistor_SMD:R_0805_2012Metric_Pad1.15x1.40mm_HandSolder, B.Cu at (168.9, 41.9)
- added R103: 330, Resistor_SMD:R_0805_2012Metric_Pad1.15x1.40mm_HandSolder, B.Cu at (106.5, 41.9)
- added R103: 330, Resistor_SMD:R_0805_2012Metric_Pad1.15x1.40mm_HandSolder, B.Cu at (44.1, 41.9)
- added R201: 120, Resistor_SMD:R_0805_2012Metric_Pad1.15x1.40mm_HandSolder, B.Cu at (245.9, 124.0)
- added R201: 120, Resistor_SMD:R_0805_2012Metric_Pad1.15x1.40mm_HandSolder, B.Cu at (183.5, 124.0)
- added R201: 120, Resistor_SMD:R_0805_2012Metric_Pad1.15x1.40mm_HandSolder, B.Cu at (121.1, 124.0)
- added R202: 4k7, Resistor_SMD:R_0805_2012Metric_Pad1.15x1.40mm_HandSolder, B.Cu at (237.6, 125.1)
- added R202: 4k7, Resistor_SMD:R_0805_2012Metric_Pad1.15x1.40mm_HandSolder, B.Cu at (175.2, 125.1)
- added R202: 4k7, Resistor_SMD:R_0805_2012Metric_Pad1.15x1.40mm_HandSolder, B.Cu at (112.8, 125.1)
- added R203: 10k, Resistor_SMD:R_0805_2012Metric_Pad1.15x1.40mm_HandSolder, B.Cu at (245.9, 111.1)
- added R203: 10k, Resistor_SMD:R_0805_2012Metric_Pad1.15x1.40mm_HandSolder, B.Cu at (183.5, 111.1)
- added R203: 10k, Resistor_SMD:R_0805_2012Metric_Pad1.15x1.40mm_HandSolder, B.Cu at (121.1, 111.1)
- added R401: 10k, Resistor_SMD:R_0805_2012Metric_Pad1.15x1.40mm_HandSolder, B.Cu at (229.4, 53.7)
- added R401: 10k, Resistor_SMD:R_0805_2012Metric_Pad1.15x1.40mm_HandSolder, B.Cu at (167.0, 53.7)
- added R401: 10k, Resistor_SMD:R_0805_2012Metric_Pad1.15x1.40mm_HandSolder, B.Cu at (104.6, 53.7)
- added R402: 1k, Resistor_SMD:R_0805_2012Metric_Pad1.15x1.40mm_HandSolder, B.Cu at (229.4, 58.8)
- added R402: 1k, Resistor_SMD:R_0805_2012Metric_Pad1.15x1.40mm_HandSolder, B.Cu at (167.0, 58.8)
- added R402: 1k, Resistor_SMD:R_0805_2012Metric_Pad1.15x1.40mm_HandSolder, B.Cu at (104.6, 58.8)
- added R403: 1k, Resistor_SMD:R_0805_2012Metric_Pad1.15x1.40mm_HandSolder, B.Cu at (229.4, 61.3)
- added R403: 1k, Resistor_SMD:R_0805_2012Metric_Pad1.15x1.40mm_HandSolder, B.Cu at (167.0, 61.3)
- added R403: 1k, Resistor_SMD:R_0805_2012Metric_Pad1.15x1.40mm_HandSolder, B.Cu at (104.6, 61.3)
- added R404: 1k, Resistor_SMD:R_0805_2012Metric_Pad1.15x1.40mm_HandSolder, B.Cu at (228.1, 91.5)
- added R404: 1k, Resistor_SMD:R_0805_2012Metric_Pad1.15x1.40mm_HandSolder, B.Cu at (165.7, 91.5)
- added R404: 1k, Resistor_SMD:R_0805_2012Metric_Pad1.15x1.40mm_HandSolder, B.Cu at (103.3, 91.5)
- added R405: 1k, Resistor_SMD:R_0805_2012Metric_Pad1.15x1.40mm_HandSolder, B.Cu at (228.1, 89.0)
- added R405: 1k, Resistor_SMD:R_0805_2012Metric_Pad1.15x1.40mm_HandSolder, B.Cu at (165.7, 89.0)
- added R405: 1k, Resistor_SMD:R_0805_2012Metric_Pad1.15x1.40mm_HandSolder, B.Cu at (103.3, 89.0)
- added R601: 330, Resistor_SMD:R_0805_2012Metric_Pad1.15x1.40mm_HandSolder, B.Cu at (231.4, 39.4)
- added R601: 330, Resistor_SMD:R_0805_2012Metric_Pad1.15x1.40mm_HandSolder, B.Cu at (169.0, 39.4)
- added R601: 330, Resistor_SMD:R_0805_2012Metric_Pad1.15x1.40mm_HandSolder, B.Cu at (106.6, 39.4)
- added R601: 330, Resistor_SMD:R_0805_2012Metric_Pad1.15x1.40mm_HandSolder, B.Cu at (44.2, 39.4)
- added TP201: SI, TestPoint:TestPoint_Pad_2.0x2.0mm, B.Cu at (249.4, 104.8)
- added TP201: SI, TestPoint:TestPoint_Pad_2.0x2.0mm, B.Cu at (187.0, 104.8)
- added TP201: SI, TestPoint:TestPoint_Pad_2.0x2.0mm, B.Cu at (124.6, 104.8)
- added TP201: SI, TestPoint:TestPoint_Pad_2.0x2.0mm, B.Cu at (62.2, 104.8)
- added TP202: SO, TestPoint:TestPoint_Pad_2.0x2.0mm, B.Cu at (249.4, 108.0)
- added TP202: SO, TestPoint:TestPoint_Pad_2.0x2.0mm, B.Cu at (187.0, 108.0)
- added TP202: SO, TestPoint:TestPoint_Pad_2.0x2.0mm, B.Cu at (124.6, 108.0)
- added TP202: SO, TestPoint:TestPoint_Pad_2.0x2.0mm, B.Cu at (62.2, 108.0)
- added TP203: TXCAN, TestPoint:TestPoint_Pad_2.0x2.0mm, B.Cu at (227.2, 115.6)
- added TP203: TXCAN, TestPoint:TestPoint_Pad_2.0x2.0mm, B.Cu at (164.8, 115.6)
- added TP203: TXCAN, TestPoint:TestPoint_Pad_2.0x2.0mm, B.Cu at (102.4, 115.6)
- added TP203: TXCAN, TestPoint:TestPoint_Pad_2.0x2.0mm, B.Cu at (40.0, 115.6)
- added TP204: RXCAN, TestPoint:TestPoint_Pad_2.0x2.0mm, B.Cu at (227.2, 111.1)
- added TP204: RXCAN, TestPoint:TestPoint_Pad_2.0x2.0mm, B.Cu at (164.8, 111.1)
- added TP204: RXCAN, TestPoint:TestPoint_Pad_2.0x2.0mm, B.Cu at (102.4, 111.1)
- added TP204: RXCAN, TestPoint:TestPoint_Pad_2.0x2.0mm, B.Cu at (40.0, 111.1)
- added TP205: SC, TestPoint:TestPoint_Pad_2.0x2.0mm, B.Cu at (249.4, 111.1)
- added TP205: SC, TestPoint:TestPoint_Pad_2.0x2.0mm, B.Cu at (187.0, 111.1)
- added TP205: SC, TestPoint:TestPoint_Pad_2.0x2.0mm, B.Cu at (124.6, 111.1)
- added TP205: SC, TestPoint:TestPoint_Pad_2.0x2.0mm, B.Cu at (62.2, 111.1)
- added TP206: SCK, TestPoint:TestPoint_Pad_2.0x2.0mm, B.Cu at (249.4, 101.6)
- added TP206: SCK, TestPoint:TestPoint_Pad_2.0x2.0mm, B.Cu at (187.0, 101.6)
- added TP206: SCK, TestPoint:TestPoint_Pad_2.0x2.0mm, B.Cu at (124.6, 101.6)
- added TP206: SCK, TestPoint:TestPoint_Pad_2.0x2.0mm, B.Cu at (62.2, 101.6)
- added TP207: CAN_H, TestPoint:TestPoint_Pad_2.0x2.0mm, B.Cu at (242.4, 123.8)
- added TP207: CAN_H, TestPoint:TestPoint_Pad_2.0x2.0mm, B.Cu at (180.0, 123.8)
- added TP207: CAN_H, TestPoint:TestPoint_Pad_2.0x2.0mm, B.Cu at (117.6, 123.8)
- added TP207: CAN_H, TestPoint:TestPoint_Pad_2.0x2.0mm, B.Cu at (55.2, 123.8)
- added TP208: CAN_L, TestPoint:TestPoint_Pad_2.0x2.0mm, B.Cu at (249.4, 123.8)
- added TP208: CAN_L, TestPoint:TestPoint_Pad_2.0x2.0mm, B.Cu at (187.0, 123.8)
- added TP208: CAN_L, TestPoint:TestPoint_Pad_2.0x2.0mm, B.Cu at (124.6, 123.8)
- added TP208: CAN_L, TestPoint:TestPoint_Pad_2.0x2.0mm, B.Cu at (62.2, 123.8)
- added TP209: INT, TestPoint:TestPoint_Pad_2.0x2.0mm, B.Cu at (243.1, 92.1)
- added TP209: INT, TestPoint:TestPoint_Pad_2.0x2.0mm, B.Cu at (180.7, 92.1)
- added TP209: INT, TestPoint:TestPoint_Pad_2.0x2.0mm, B.Cu at (118.3, 92.1)
- added TP209: INT, TestPoint:TestPoint_Pad_2.0x2.0mm, B.Cu at (55.9, 92.1)
- added U201: MCP2551-I/SN, Package_SO:SOIC-8_3.9x4.9mm_P1.27mm, B.Cu at (237.6, 117.9)
- added U201: MCP2551-I/SN, Package_SO:SOIC-8_3.9x4.9mm_P1.27mm, B.Cu at (175.2, 117.9)
- added U201: MCP2551-I/SN, Package_SO:SOIC-8_3.9x4.9mm_P1.27mm, B.Cu at (112.8, 117.9)
- added U202: MCP2515-xSO, Package_SO:SOIC-18W_7.5x11.6mm_P1.27mm, B.Cu at (237.6, 105.8)
- added U202: MCP2515-xSO, Package_SO:SOIC-18W_7.5x11.6mm_P1.27mm, B.Cu at (175.2, 105.8)
- added U202: MCP2515-xSO, Package_SO:SOIC-18W_7.5x11.6mm_P1.27mm, B.Cu at (112.8, 105.8)
- added U301: A1101ELHL, Package_TO_SOT_SMD:SOT-23, B.Cu at (239.9, 43.5)
- added U301: A1101ELHL, Package_TO_SOT_SMD:SOT-23, B.Cu at (177.5, 43.5)
- added U301: A1101ELHL, Package_TO_SOT_SMD:SOT-23, B.Cu at (115.1, 43.5)
- added U401: ATMEGA328P-PU, Package_DIP:DIP-28_W7.62mm_Socket, F.Cu at (234.4, 56.3)
- added U401: ATMEGA328P-PU, Package_DIP:DIP-28_W7.62mm_Socket, F.Cu at (172.0, 56.3)
- added U401: ATMEGA328P-PU, Package_DIP:DIP-28_W7.62mm_Socket, F.Cu at (109.6, 56.3)
- added U501: LM7805, KicadZeniteSolarLibrary18:TO-220-3_Horizontal_TabDown_SMD, B.Cu at (257.1, 89.5)
- added U501: LM7805, KicadZeniteSolarLibrary18:TO-220-3_Horizontal_TabDown_SMD, B.Cu at (194.7, 89.5)
- added U501: LM7805, KicadZeniteSolarLibrary18:TO-220-3_Horizontal_TabDown_SMD, B.Cu at (132.2, 89.5)
- added Y201: 16MHz, Crystal:Crystal_HC49-U_Vertical, F.Cu at (226.8, 105.8)
- added Y201: 16MHz, Crystal:Crystal_HC49-U_Vertical, F.Cu at (164.4, 105.8)
- added Y201: 16MHz, Crystal:Crystal_HC49-U_Vertical, F.Cu at (102.0, 105.8)
- added Y401: 16MHz, Crystal:Crystal_HC49-U_Vertical, F.Cu at (228.1, 81.7)
- added Y401: 16MHz, Crystal:Crystal_HC49-U_Vertical, F.Cu at (165.7, 81.7)
- added Y401: 16MHz, Crystal:Crystal_HC49-U_Vertical, F.Cu at (103.3, 81.7)
- added Z101: 4.7V, Diode_SMD:D_MiniMELF_Handsoldering, B.Cu at (235.5, 45.9)
- added Z101: 4.7V, Diode_SMD:D_MiniMELF_Handsoldering, B.Cu at (173.1, 45.9)
- added Z101: 4.7V, Diode_SMD:D_MiniMELF_Handsoldering, B.Cu at (110.7, 45.9)
- added Z102: 4.7V, Diode_SMD:D_MiniMELF_Handsoldering, B.Cu at (242.7, 47.6)
- added Z102: 4.7V, Diode_SMD:D_MiniMELF_Handsoldering, B.Cu at (180.3, 47.6)
- added Z102: 4.7V, Diode_SMD:D_MiniMELF_Handsoldering, B.Cu at (117.9, 47.6)
- R101: value 100 -> 330
- moved R101 31.3 mm to (44.1, 44.5)
- moved J1 31.3 mm to (67.9, 38.7)
- moved C1 31.0 mm to (51.8, 50.8)
- moved C201 31.0 mm to (47.6, 97.2)
- moved C204 31.0 mm to (42.2, 99.4)
- moved C205 31.0 mm to (50.4, 122.9)
- moved C402 31.0 mm to (43.4, 71.5)
- moved C404 31.0 mm to (42.2, 74.7)
- moved C405 31.0 mm to (42.2, 56.3)
- moved C406 31.0 mm to (44.6, 51.3)
- moved C501 31.0 mm to (70.7, 99.1)
- moved C504 31.0 mm to (64.2, 95.2)
- moved D101 31.0 mm to (41.5, 47.6)
- moved D501 31.0 mm to (76.2, 112.4)
- moved F501 31.0 mm to (76.2, 103.5)
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Routing:
- net +5V: track 202.9 -> 837.0 mm
- net GND: track 82.6 -> 390.2 mm, vias 14 -> 64
- net /POWER SUPPLY/+18V_IN: track 71.9 -> 287.8 mm
- net /CANBUS CONN/CAN_H: track 50.6 -> 212.5 mm
- net /CANBUS CONN/CAN_L: track 48.2 -> 205.5 mm, vias 2 -> 8
- net /MISO: track 37.7 -> 150.9 mm
- net /MCU/VOUT: track 33.8 -> 145.6 mm
- net /SCK: track 35.6 -> 142.3 mm
- net /MOSI: track 32.9 -> 131.5 mm
- net /CANBUS/CS: track 32.2 -> 128.6 mm
- net /MCU/SDA: track 25.2 -> 103.0 mm
- net /MCU/SCL: track 22.0 -> 90.1 mm
- net /CANBUS/INT: track 21.1 -> 85.0 mm
- net Net-(C101-Pad1): track 9.59 -> 67.7 mm
- net /CANBUS/TXCAN: track 15.4 -> 65.8 mm
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Other:
- board size 52.1 x 121.3 mm -> 239.3 x 121.3 mm
