File: hardware/basicsensormodule.kicad_pcb (KiCad board)
At the start: 2 copper layers, 239.3 x 121.3 mm, 252 parts, among them J1 Conn_01x04, J401 USART, J601 RJ45, J602 RJ45, U201 MCP2551-I/SN, U202 MCP2515-xSO, U301 A1101ELHL, U401 ATMEGA328P-PU, U501 LM7805, Y201 16MHz, Y401 16MHz

Commit message: 3D exported
Parts:
- removed the C1 at (176.6, 50.8)
- removed the C1 at (114.2, 50.8)
- removed the C1 at (51.8, 50.8)
- removed the C101 at (172.8, 39.4)
- removed the C101 at (110.4, 39.4)
- removed the C101 at (48.0, 39.4)
- removed the C102 at (186.2, 41.9)
- removed the C102 at (123.8, 41.9)
- removed the C102 at (61.4, 41.9)
- removed the C201 at (172.4, 97.2)
- removed the C201 at (110.0, 97.2)
- removed the C201 at (47.6, 97.2)
- removed the C202 at (180.0, 113.0)
- removed the C202 at (117.6, 113.0)
- removed the C202 at (55.2, 113.0)
- removed the C203 at (164.8, 103.3)
- removed the C203 at (102.4, 103.3)
- removed the C203 at (40.0, 103.3)
- removed the C204 at (167.0, 99.4)
- removed the C204 at (104.6, 99.4)
- removed the C204 at (42.2, 99.4)
- removed the C205 at (175.2, 122.9)
- removed the C205 at (112.8, 122.9)
- removed the C205 at (50.4, 122.9)
- removed the C401 at (183.5, 76.6)
- removed the C401 at (121.1, 76.6)
- removed the C401 at (58.7, 76.6)
- removed the C402 at (168.2, 71.5)
- removed the C402 at (105.8, 71.5)
- removed the C402 at (43.4, 71.5)
- removed the C403 at (165.7, 79.1)
- removed the C403 at (103.3, 79.1)
- removed the C403 at (40.9, 79.1)
- removed the C404 at (167.0, 74.7)
- removed the C404 at (104.6, 74.7)
- removed the C404 at (42.2, 74.7)
- removed the C405 at (167.0, 56.3)
- removed the C405 at (104.6, 56.3)
- removed the C405 at (42.2, 56.3)
- removed the C406 at (169.4, 51.3)
- removed the C406 at (107.0, 51.3)
- removed the C406 at (44.6, 51.3)
- removed the C501 at (195.5, 99.1)
- removed the C501 at (133.1, 99.1)
- removed the C501 at (70.7, 99.1)
- removed the C502 at (195.5, 95.2)
- removed the C502 at (133.1, 95.2)
- removed the C502 at (70.7, 95.2)
- removed the C503 at (188.9, 98.4)
- removed the C503 at (126.5, 98.4)
- removed the C503 at (64.1, 98.4)
- removed the C504 at (189.0, 95.2)
- removed the C504 at (126.6, 95.2)
- removed the C504 at (64.2, 95.2)
- removed the D101 at (166.3, 47.6)
- removed the D101 at (103.9, 47.6)
- removed the D101 at (41.5, 47.6)
- removed the D201 at (183.5, 128.0)
- removed the D201 at (121.1, 128.0)
- removed the D201 at (58.7, 128.0)
- removed the D401 at (162.4, 51.4)
- removed the D401 at (100.0, 51.4)
- removed the D401 at (37.6, 51.4)
- removed the D402 at (161.9, 91.5)
- removed the D402 at (99.5, 91.5)
- removed the D402 at (37.1, 91.5)
- removed the D403 at (161.9, 89.0)
- removed the D403 at (99.5, 89.0)
- removed the D403 at (37.1, 89.0)
- removed the D501 at (201.0, 112.4)
- removed the D501 at (138.6, 112.4)
- removed the D501 at (76.2, 112.4)
- removed the F501 at (201.0, 103.5)
- removed the F501 at (138.6, 103.5)
- removed the F501 at (76.2, 103.5)
- removed the H101 at (159.7, 40.6)
- removed the H101 at (97.3, 40.6)
- removed the H101 at (34.9, 40.6)
- removed the H102 at (159.3, 126.1)
- removed the H102 at (96.9, 126.1)
- removed the H102 at (34.5, 126.1)
- removed the H103 at (201.6, 125.1)
- removed the H103 at (139.2, 125.1)
- removed the H103 at (76.8, 125.1)
- removed the H104 at (201.6, 40.6)
- removed the H104 at (139.2, 40.6)
- removed the H104 at (76.8, 40.6)
- removed the J1 at (192.7, 38.7)
- removed the J1 at (130.3, 38.7)
- removed the J1 at (67.9, 38.7)
- removed the J401 at (159.3, 63.9)
- removed the J401 at (96.9, 63.9)
- removed the J401 at (34.5, 63.9)
- removed the J601 at (186.0, 138.8)
- removed the J601 at (123.6, 138.8)
- removed the J601 at (61.2, 138.8)
- removed the J602 at (165.2, 138.8)
- removed the J602 at (102.8, 138.8)
- removed the J602 at (40.4, 138.8)
- removed the R101 at (168.9, 44.5)
- removed the R101 at (106.5, 44.5)
- removed the R101 at (44.1, 44.5)
- removed the R102 at (177.5, 40.0)
- removed the R102 at (115.1, 40.0)
- removed the R102 at (52.7, 40.0)
- removed the R103 at (168.9, 41.9)
- removed the R103 at (106.5, 41.9)
- removed the R103 at (44.1, 41.9)
- removed the R201 at (183.5, 124.0)
- removed the R201 at (121.1, 124.0)
- removed the R201 at (58.7, 124.0)
- removed the R202 at (175.2, 125.1)
- removed the R202 at (112.8, 125.1)
- removed the R202 at (50.4, 125.1)
- removed the R203 at (183.5, 111.1)
- removed the R203 at (121.1, 111.1)
- removed the R203 at (58.7, 111.1)
- removed the R401 at (167.0, 53.7)
- removed the R401 at (104.6, 53.7)
- removed the R401 at (42.2, 53.7)
- removed the R402 at (167.0, 58.8)
- removed the R402 at (104.6, 58.8)
- removed the R402 at (42.2, 58.8)
- removed the R403 at (167.0, 61.3)
- removed the R403 at (104.6, 61.3)
- removed the R403 at (42.2, 61.3)
- removed the R404 at (165.7, 91.5)
- removed the R404 at (103.3, 91.5)
- removed the R404 at (40.9, 91.5)
- removed the R405 at (165.7, 89.0)
- removed the R405 at (103.3, 89.0)
- removed the R405 at (40.9, 89.0)
- removed the R601 at (169.0, 39.4)
- removed the R601 at (106.6, 39.4)
- removed the R601 at (44.2, 39.4)
- removed the TP201 at (187.0, 104.8)
- removed the TP201 at (124.6, 104.8)
- removed the TP201 at (62.2, 104.8)
- removed the TP202 at (187.0, 108.0)
- removed the TP202 at (124.6, 108.0)
- removed the TP202 at (62.2, 108.0)
- removed the TP203 at (164.8, 115.6)
- removed the TP203 at (102.4, 115.6)
- removed the TP203 at (40.0, 115.6)
- removed the TP204 at (164.8, 111.1)
- removed the TP204 at (102.4, 111.1)
- removed the TP204 at (40.0, 111.1)
- removed the TP205 at (187.0, 111.1)
- removed the TP205 at (124.6, 111.1)
- removed the TP205 at (62.2, 111.1)
- removed the TP206 at (187.0, 101.6)
- removed the TP206 at (124.6, 101.6)
- removed the TP206 at (62.2, 101.6)
- removed the TP207 at (180.0, 123.8)
- removed the TP207 at (117.6, 123.8)
- removed the TP207 at (55.2, 123.8)
- removed the TP208 at (187.0, 123.8)
- removed the TP208 at (124.6, 123.8)
- removed the TP208 at (62.2, 123.8)
- removed the TP209 at (180.7, 92.1)
- removed the TP209 at (118.3, 92.1)
- removed the TP209 at (55.9, 92.1)
- removed the U201 at (175.2, 117.9)
- removed the U201 at (112.8, 117.9)
- removed the U201 at (50.4, 117.9)
- removed the U202 at (175.2, 105.8)
- removed the U202 at (112.8, 105.8)
- removed the U202 at (50.4, 105.8)
- removed the U301 at (177.5, 43.5)
- removed the U301 at (115.1, 43.5)
- removed the U301 at (52.7, 43.5)
- removed the U401 at (172.0, 56.3)
- removed the U401 at (109.6, 56.3)
- removed the U401 at (47.2, 56.3)
- removed the U501 at (194.7, 89.5)
- removed the U501 at (132.2, 89.5)
- removed the U501 at (69.8, 89.5)
- removed the Y201 at (164.4, 105.8)
- removed the Y201 at (102.0, 105.8)
- removed the Y201 at (39.6, 105.8)
- removed the Y401 at (165.7, 81.7)
- removed the Y401 at (103.3, 81.7)
- removed the Y401 at (40.9, 81.7)
- removed the Z101 at (173.1, 45.9)
- removed the Z101 at (110.7, 45.9)
- removed the Z101 at (48.3, 45.9)
- removed the Z102 at (180.3, 47.6)
- removed the Z102 at (117.9, 47.6)
- removed the Z102 at (55.5, 47.6)
- moved H104 174.5 mm to (93.4, 77.2), turned to 0 degrees
- moved J1 170.4 mm to (91.5, 86.1), turned to 0 degrees
- moved C102 162.1 mm to (94.7, 92.7), turned to 90 degrees
- moved R102 159.4 mm to (92.8, 101.3), turned to 90 degrees
- moved C101 157.9 mm to (92.1, 106.0), turned to 90 degrees
- moved R601 156.1 mm to (92.1, 109.8), turned to 270 degrees
- moved U301 154.8 mm to (96.3, 101.3), turned to 0 degrees
- moved R103 152.6 mm to (94.7, 110.0), turned to 90 degrees
- moved Z102 151.1 mm to (100.4, 98.6), turned to 270 degrees
- moved H101 150.8 mm to (93.4, 119.1), turned to 0 degrees
- moved Z101 149.3 mm to (98.7, 105.8), turned to 0 degrees
- moved R101 149.2 mm to (97.2, 110.0), turned to 270 degrees
- moved C1 144.9 mm to (103.5, 102.2), turned to 270 degrees
- moved D101 143.8 mm to (100.4, 112.6), turned to 270 degrees
- moved C406 140.3 mm to (104.1, 109.5), turned to 270 degrees
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Routing:
- net +5V: track 837.0 -> 209.3 mm
- net GND: track 390.2 -> 97.6 mm, vias 64 -> 16
- net /POWER SUPPLY/+18V_IN: track 287.8 -> 71.9 mm
- net /CANBUS CONN/CAN_H: track 212.5 -> 53.1 mm
- net /CANBUS CONN/CAN_L: track 205.5 -> 51.4 mm, vias 8 -> 2
- net /MISO: track 150.9 -> 37.7 mm
- net /MCU/VOUT: track 145.6 -> 36.4 mm
- net /SCK: track 142.3 -> 35.6 mm
- net /MOSI: track 131.5 -> 32.9 mm
- net /CANBUS/CS: track 128.6 -> 32.2 mm
- net /MCU/SDA: track 103.0 -> 25.7 mm
- net /MCU/SCL: track 90.1 -> 22.5 mm
- net /CANBUS/INT: track 85.0 -> 21.3 mm
- net Net-(C101-Pad1): track 67.7 -> 16.9 mm
- net /CANBUS/TXCAN: track 65.8 -> 16.5 mm
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Other:
- board size 239.3 x 121.3 mm -> 121.3 x 52.1 mm
