File: hardware/hall_effect_sensor.sch (KiCad schematic (older format))
At the start: 8 parts, among them U301 A1101ELHL

Commit message: layout finalizado
Parts:
- added R103, R601: 330, Resistor_SMD:R_0805_2012Metric_Pad1.15x1.40mm_HandSolder, symbol Device:R_Small
- R101: value 100 -> 330
Connections:
- net at C101.1, R101.1, R102.1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: now also R103.1, R601.1
- net at D101.1 (K), R101.2: now also R103.2, R601.2
Other:
- moved on the sheet: D101
Changed lines of the file:
@@
 AR Path="/5CD559BA/5CD661DC" Ref="R101"  Part="1"
 F 0 "R101" V 3754 2450 50  0000 C CNN
-F 1 "100" V 3845 2450 50  0000 C CNN
+F 1 "330" V 3845 2450 50  0000 C CNN
 F 2 "Resistor_SMD:R_0805_2012Metric_Pad1.15x1.40mm_HandSolder" H 3950 2450 50  0001 C CNN
 F 3 "~" H 3950 2450 50  0001 C CNN
@@
 L Device:D_Small D?
 U 1 1 5CD661F4
-P 3650 2450
+P 3000 2450
 AR Path="/5CD661F4" Ref="D?"  Part="1"
 AR Path="/5CD559BA/5CD661F4" Ref="D101"  Part="1"
-F 0 "D101" H 3650 2245 50  0000 C CNN
-F 1 "LL4148" H 3650 2336 50  0000 C CNN
-F 2 "Diode_SMD:D_MiniMELF_Handsoldering" V 3650 2450 50  0001 C CNN
-F 3 "~" V 3650 2450 50  0001 C CNN
-	1    3650 2450
+F 0 "D101" H 3000 2245 50  0000 C CNN
+F 1 "LL4148" H 3000 2336 50  0000 C CNN
+F 2 "Diode_SMD:D_MiniMELF_Handsoldering" V 3000 2450 50  0001 C CNN
+F 3 "~" V 3000 2450 50  0001 C CNN
+	1    3000 2450
 	-1   0    0    1
 $EndComp
 Wire Wire Line
-	3750 2450 3850 2450
-Wire Wire Line
 	4050 2450 4300 2450
 Wire Wire Line
 	6400 2450 6400 2500
-Wire Wire Line
-	4300 2800 4300 2450
 Connection ~ 4300 2450
 Wire Wire Line
@@
 L power:+5V #PWR?
 U 1 1 5CD6621D
-P 3450 2400
+P 2250 2450
 AR Path="/5CD6621D" Ref="#PWR?"  Part="1"
 AR Path="/5CD559BA/5CD6621D" Ref="#PWR0112"  Part="1"
-F 0 "#PWR0112" H 3450 2250 50  0001 C CNN
-F 1 "+5V" H 3465 2573 50  0000 C CNN
-F 2 "" H 3450 2400 50  0001 C CNN
-F 3 "" H 3450 2400 50  0001 C CNN
-	1    3450 2400
+F 0 "#PWR0112" H 2250 2300 50  0001 C CNN
+F 1 "+5V" H 2265 2623 50  0000 C CNN
+F 2 "" H 2250 2450 50  0001 C CNN
+F 3 "" H 2250 2450 50  0001 C CNN
+	1    2250 2450
 	1    0    0    -1
 $EndComp
@@
 L power:+5V #PWR?
 U 1 1 5CD6D8F6
-P 3950 2850
+P 3100 2800
 AR Path="/5CD6D8F6" Ref="#PWR?"  Part="1"
 AR Path="/5CD559BA/5CD6D8F6" Ref="#PWR0113"  Part="1"
-F 0 "#PWR0113" H 3950 2700 50  0001 C CNN
-F 1 "+5V" H 3965 3023 50  0000 C CNN
-F 2 "" H 3950 2850 50  0001 C CNN
-F 3 "" H 3950 2850 50  0001 C CNN
-	1    3950 2850
+F 0 "#PWR0113" H 3100 2650 50  0001 C CNN
+F 1 "+5V" H 3115 2973 50  0000 C CNN
+F 2 "" H 3100 2800 50  0001 C CNN
+F 3 "" H 3100 2800 50  0001 C CNN
+	1    3100 2800
 	1    0    0    -1
 $EndComp
@@
 L power:GND #PWR?
 U 1 1 5CD6DFF4
-P 3950 3100
+P 3100 3050
 AR Path="/5CD6DFF4" Ref="#PWR?"  Part="1"
 AR Path="/5CD559BA/5CD6DFF4" Ref="#PWR0114"  Part="1"
-F 0 "#PWR0114" H 3950 2850 50  0001 C CNN
-F 1 "GND" H 3955 2927 50  0000 C CNN
-F 2 "" H 3950 3100 50  0001 C CNN
-F 3 "" H 3950 3100 50  0001 C CNN
-	1    3950 3100
-	1    0    0    -1
-$EndComp
-Text HLabel 3750 2850 0    50   Input ~ 0
+F 0 "#PWR0114" H 3100 2800 50  0001 C CNN
+F 1 "GND" H 3105 2877 50  0000 C CNN
+F 2 "" H 3100 3050 50  0001 C CNN
+F 3 "" H 3100 3050 50  0001 C CNN
+	1    3100 3050
+	1    0    0    -1
+$EndComp
+Text HLabel 2900 2800 0    50   Input ~ 0
 VCC
 Wire Wire Line
-	3750 2850 3950 2850
-Text HLabel 3750 3100 0    50   Output ~ 0
+	2900 2800 3100 2800
+Text HLabel 2900 3050 0    50   Output ~ 0
 GND
 Wire Wire Line
-	3750 3100 3950 3100
-Wire Wire Line
-	3550 2450 3450 2450
-Wire Wire Line
-	3450 2450 3450 2400
+	2900 3050 3100 3050
 Text HLabel 7400 2950 2    50   Output ~ 0
 VOUT
@@
 Wire Wire Line
 	6400 3500 6400 3400
+$Comp
+L Device:R_Small R601
+U 1 1 5CDE1807
+P 3950 2050
+F 0 "R601" V 3754 2050 50  0000 C CNN
+F 1 "330" V 3845 2050 50  0000 C CNN
+F 2 "Resistor_SMD:R_0805_2012Metric_Pad1.15x1.40mm_HandSolder" H 3950 2050 50  0001 C CNN
+F 3 "~" H 3950 2050 50  0001 C CNN
+	1    3950 2050
+	0    1    1    0
+$EndComp
+Wire Wire Line
+	4300 2800 4300 2750
+Wire Wire Line
+	4300 2450 4300 2050
+Wire Wire Line
+	4300 2050 4050 2050
+Wire Wire Line
+	2900 2450 2250 2450
+Wire Wire Line
+	3100 2450 3600 2450
+Wire Wire Line
+	3850 2050 3600 2050
+Wire Wire Line
+	3600 2050 3600 2450
+Connection ~ 3600 2450
+Wire Wire Line
+	3600 2450 3850 2450
+$Comp
+L Device:R_Small R103
+U 1 1 5CDE6DF6
+P 3950 2750
+F 0 "R103" V 3754 2750 50  0000 C CNN
+F 1 "330" V 3845 2750 50  0000 C CNN
+F 2 "Resistor_SMD:R_0805_2012Metric_Pad1.15x1.40mm_HandSolder" H 3950 2750 50  0001 C CNN
+F 3 "~" H 3950 2750 50  0001 C CNN
+	1    3950 2750
+	0    1    1    0
+$EndComp
+Wire Wire Line
+	4050 2750 4300 2750
+Connection ~ 4300 2750
+Wire Wire Line
+	4300 2750 4300 2450
+Wire Wire Line
+	3850 2750 3600 2750
+Wire Wire Line
+	3600 2750 3600 2450
 $EndSCHEMATC
